File: Amplifier.kicad_pcb (KiCad board)
At the start: 2 copper layers, 55.4 x 27.7 mm, 22 parts, among them Q1 BC547, Q2 2N3904

Commit message: 2.26.2026
Parts:
- moved Q2 10.2 mm to (111.2, 55.8)
- moved Q1 10.2 mm to (96.7, 53.3)
- moved C3 8.92 mm to (97.0, 61.6)
- moved C5 8.28 mm to (112.5, 66.7)
- moved C6 8.28 mm to (108.9, 66.7)
Routing:
- net Net-(Q2-C): track 17.4 -> 27.1 mm
- net Net-(Q1-E): track 5.29 -> 13.3 mm
- net Net-(Q1-B): track 28.9 -> 21.1 mm
- net Net-(Q2-B): track 39.6 -> 32.4 mm
- net Net-(Q2-E): track 6.56 -> 13.4 mm
- net Net-(C5-Pad1): track 10.1 -> 16.6 mm
- added copper zone on B.Cu, net (none)
Changed lines of the file:
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@@
 	(paper "A5")
 	(title_block
-		(title "Power_Amplifier")
+		(title "Amplifier")
 	)
 	(layers
@@
 	(footprint "Capacitor_THT:C_Disc_D5.1mm_W3.2mm_P5.00mm"
 		(layer "F.Cu")
-		(at 97.01 52.717 -90)
+		(at 97.028 61.635 -90)
 		(descr "C, Disc series, Radial, pin pitch=5.00mm, diameter*width=5.1*3.2mm^2, Capacitor, http://www.vishay.com/docs/45233/krseries.pdf")
 		(tags "C Disc series Radial pin pitch 5.00mm diameter 5.1mm width 3.2mm Capacitor")
@@
 	(footprint "Package_TO_SOT_THT:TO-92_Inline"
 		(layer "F.Cu")
-		(at 96.7 63.497 -90)
+		(at 96.668 53.34 -90)
 		(descr "TO-92 leads in-line, narrow, oval pads, drill 0.75mm (see NXP sot054_po.pdf)")
 		(tags "to-92 sc-43 sc-43a sot54 PA33 transistor")
@@
 	(footprint "Capacitor_THT:C_Disc_D5.1mm_W3.2mm_P5.00mm"
 		(layer "F.Cu")
-		(at 112.522 58.38 90)
+		(at 112.54 66.663 90)
 		(descr "C, Disc series, Radial, pin pitch=5.00mm, diameter*width=5.1*3.2mm^2, Capacitor, http://www.vishay.com/docs/45233/krseries.pdf")
 		(tags "C Disc series Radial pin pitch 5.00mm diameter 5.1mm width 3.2mm Capacitor")
@@
 	(footprint "Package_TO_SOT_THT:TO-92_Inline"
 		(layer "F.Cu")
-		(at 111.2 65.992 90)
+		(at 111.168 55.835 90)
 		(descr "TO-92 leads in-line, narrow, oval pads, drill 0.75mm (see NXP sot054_po.pdf)")
 		(tags "to-92 sc-43 sc-43a sot54 PA33 transistor")
@@
 	(footprint "Capacitor_THT:C_Disc_D4.3mm_W1.9mm_P5.00mm"
 		(layer "F.Cu")
-		(at 108.839 58.38 90)
+		(at 108.857 66.663 90)
 		(descr "C, Disc series, Radial, pin pitch=5.00mm, diameter*width=4.3*1.9mm^2, Capacitor, http://www.vishay.com/docs/45233/krseries.pdf")
 		(tags "C Disc series Radial pin pitch 5.00mm diameter 4.3mm width 1.9mm Capacitor")
@@
 	)
 	(segment
-		(start 92.062 67.564)
-		(end 98.552 67.564)
-		(width 1)
-		(layer "B.Cu")
-		(net 4)
-	)
-	(segment
 		(start 88.585 61.6245)
 		(end 88.6125 61.597)
@@
 	)
 	(segment
-		(start 99.568 65.405)
-		(end 98.93 64.767)
-		(width 1)
-		(layer "B.Cu")
-		(net 4)
-	)
-	(segment
-		(start 88.585 64.087)
-		(end 92.062 67.564)
-		(width 1)
+		(start 96.668 54.61)
+		(end 91.683 54.61)
+		(width 0.85)
 		(layer "B.Cu")
 		(net 4)
 	)
 	(segment
-		(start 98.552 67.564)
-		(end 99.568 66.548)
-		(width 1)
-		(layer "B.Cu")
-		(net 4)
-	)
-	(segment
-		(start 99.568 66.548)
-		(end 99.568 65.405)
-		(width 1)
-		(layer "B.Cu")
-		(net 4)
-	)
-	(segment
-		(start 98.93 64.767)
-		(end 96.7 64.767)
-		(width 1)
+		(start 91.683 54.61)
+		(end 88.6125 57.6805)
+		(width 0.85)
 		(layer "B.Cu")
 		(net 4)
@@
 	)
 	(segment
+		(start 113.665 56.855)
+		(end 113.665 55.372)
+		(width 0.85)
+		(layer "B.Cu")
+		(net 6)
+	)
+	(segment
 		(start 101.785 61.672)
 		(end 101.7175 61.6045)
@@
 	)
 	(segment
-		(start 113.363 64.722)
-		(end 111.2 64.722)
-		(width 1)
+		(start 101.785 60.54063)
+		(end 101.785 61.672)
+		(width 0.85)
 		(layer "B.Cu")
 		(net 6)
 	)
 	(segment
-		(start 97.01 57.717)
-		(end 97.83 57.717)
-		(width 1)
+		(start 111.168 54.565)
+		(end 107.76063 54.565)
+		(width 0.85)
 		(layer "B.Cu")
 		(net 6)
 	)
 	(segment
-		(start 114.3 67.31)
-		(end 114.3 65.659)
-		(width 1)
+		(start 107.76063 54.565)
+		(end 101.785 60.54063)
+		(width 0.85)
 		(layer "B.Cu")
 		(net 6)
 	)
 	(segment
-		(start 97.83 57.717)
-		(end 101.785 61.672)
+		(start 97.028 66.635)
+		(end 99.237 66.635)
 		(width 1)
 		(layer "B.Cu")
@@
 	)
 	(segment
-		(start 114.3 65.659)
-		(end 113.363 64.722)
+		(start 99.237 66.635)
+		(end 101.81 64.062)
 		(width 1)
 		(layer "B.Cu")
@@
 	)
 	(segment
-		(start 101.7175 61.6045)
-		(end 101.7175 60.5015)
-		(width 1)
+		(start 108.857 61.663)
+		(end 113.665 56.855)
+		(width 0.85)
 		(layer "B.Cu")
 		(net 6)
 	)
 	(segment
-		(start 101.81 64.062)
-		(end 105.693 67.945)
+		(start 101.81 61.697)
+		(end 101.785 61.672)
 		(width 1)
 		(layer "B.Cu")
@@
 	)
 	(segment
-		(start 101.81 61.697)
-		(end 101.785 61.672)
-		(width 1)
+		(start 113.665 55.372)
+		(end 112.858 54.565)
+		(width 0.85)
 		(layer "B.Cu")
 		(net 6)
 	)
 	(segment
-		(start 101.7175 60.5015)
-		(end 108.839 53.38)
-		(width 1)
+		(start 112.858 54.565)
+		(end 111.168 54.565)
+		(width 0.85)
 		(layer "B.Cu")
 		(net 6)
 	)
 	(segment
-		(start 113.665 67.945)
-		(end 114.3 67.31)
+		(start 98.015 53.184)
+		(end 96.668 53.184)
 		(width 1)
 		(layer "B.Cu")
-		(net 6)
+		(net 7)
 	)
 	(segment
-		(start 105.693 67.945)
-		(end 113.665 67.945)
+		(start 99.187 59.69)
+		(end 99.187 54.356)
 		(width 1)
 		(layer "B.Cu")
-		(net 6)
+		(net 7)
 	)
 	(segment
-		(start 94.85 61.647)
-		(end 96.7 63.497)
+		(start 92.21 61.647)
+		(end 97.016 61.647)
 		(width 1)
 		(layer "B.Cu")
@@
 	)
 	(segment
-		(start 92.21 61.647)
-		(end 94.85 61.647)
+		(start 97.016 61.647)
+		(end 97.028 61.635)
 		(width 1)
 		(layer "B.Cu")
@@
 	)
 	(segment
-		(start 92.21 57.517)
-		(end 97.01 52.717)
+		(start 99.187 54.356)
+		(end 98.015 53.184)
 		(width 1)
 		(layer "B.Cu")
@@
 	)
 	(segment
-		(start 92.21 61.647)
-		(end 92.21 57.517)
+		(start 97.242 61.635)
+		(end 99.187 59.69)
+		(width 1)
+		(layer "B.Cu")
+		(net 7)
+	)
+	(segment
+		(start 97.028 61.635)
+		(end 97.242 61.635)
 		(width 1)
 		(layer "B.Cu")
@@
 	)
 	(segment
-		(start 108.839 58.38)
-		(end 108.839 57.063)
+		(start 114.734 53.139)
+		(end 111.168 53.139)
 		(width 1)
 		(layer "B.Cu")
@@
 	)
 	(segment
-		(start 105.522 61.697)
-		(end 108.839 58.38)
+		(start 108.857 66.663)
+		(end 108.857 65.346)
 		(width 1)
 		(layer "B.Cu")
@@
 	)
 	(segment
-		(start 108.839 58.38)
-		(end 108.839 61.091)
+		(start 108.857 65.144)
+		(end 105.41 61.697)
 		(width 1)
 		(layer "B.Cu")
@@
 	)
 	(segment
-		(start 108.839 57.063)
-		(end 112.522 53.38)
+		(start 108.857 66.663)
+		(end 108.857 65.144)
 		(width 1)
 		(layer "B.Cu")
@@
 	)
 	(segment
-		(start 108.839 61.091)
-		(end 111.2 63.452)
+		(start 108.857 65.346)
+		(end 112.54 61.663)
 		(width 1)
 		(layer "B.Cu")
@@
 	)
 	(segment
-		(start 112.522 58.38)
-		(end 115.5685 58.38)
+		(start 112.54 61.663)
+		(end 112.708 61.663)
+		(width 1)
+		(layer "B.Cu")
+		(net 9)
+	)
+	(segment
+		(start 115.951 54.356)
+		(end 114.734 53.139)
+		(width 1)
+		(layer "B.Cu")
+		(net 9)
+	)
+	(segment
+		(start 115.951 58.42)
+		(end 115.951 54.356)
+		(width 1)
+		(layer "B.Cu")
+		(net 9)
+	)
+	(segment
+		(start 112.708 61.663)
+		(end 115.951 58.42)
+		(width 1)
+		(layer "B.Cu")
+		(net 9)
+	)
+	(segment
+		(start 112.54 65.26)
+		(end 117.856 59.944)
 		(width 1)
 		(layer "B.Cu")
@@
 	)
 	(segment
-		(start 115.5685 58.38)
+		(start 117.856 56.0925)
 		(end 120.5685 53.38)
 		(width 1)
@@
 	)
 	(segment
+		(start 117.856 59.944)
+		(end 117.856 56.0925)
+		(width 1)
+		(layer "B.Cu")
+		(net 10)
+	)
+	(segment
+		(start 112.54 66.663)
+		(end 112.54 65.26)
+		(width 1)
+		(layer "B.Cu")
+		(net 10)
+	)
+	(segment
+		(start 93.443 56.036)
+		(end 96.668 56.036)
+		(width 1)
+		(layer "B.Cu")
+		(net 11)
+	)
+	(segment
 		(start 92.185 64.162)
-		(end 94.06 66.037)
+		(end 90.424 62.401)
 		(width 1)
 		(layer "B.Cu")
@@
 	)
 	(segment
-		(start 94.06 66.037)
-		(end 96.7 66.037)
+		(start 90.424 62.401)
+		(end 90.424 59.055)
 		(width 1)
 		(layer "B.Cu")
@@
 	)
 	(segment
-		(start 107.265 65.992)
-		(end 111.2 65.992)
+		(start 90.424 59.055)
+		(end 93.443 56.036)
+		(width 1)
+		(layer "B.Cu")
+		(net 11)
+	)
+	(segment
+		(start 108.710422 55.991)
+		(end 111.168 55.991)
+		(width 1)
+		(layer "B.Cu")
+		(net 12)
+	)
+	(segment
+		(start 103.709 62.436)
+		(end 103.709 60.992422)
 		(width 1)
 		(layer "B.Cu")
@@
 	(segment
 		(start 105.41 64.137)
-		(end 107.265 65.992)
+		(end 103.709 62.436)
+		(width 1)
+		(layer "B.Cu")
+		(net 12)
+	)
+	(segment
+		(start 103.709 60.992422)
+		(end 108.710422 55.991)
 		(width 1)
 		(layer "B.Cu")
@@
 		(net 13)
 	)
+	(zone
+		(net 0)
+		(net_name "")
+		(layer "B.Cu")
+		(hatch edge 0.5)
+		(connect_pads
+			(clearance 0.5)
+		)
+		(min_thickness 0.25)
+		(filled_areas_thickness no)
+		(fill yes
+			(thermal_gap 0.5)
+			(thermal_bridge_width 0.5)
+			(island_removal_mode 1)
+			(island_area_min 10)
+		)
+		(polygon
+			(pts
+				(xy 71.0184 49.4284) (xy 71.0184 77.1144) (xy 126.3904 77.1144) (xy 126.3904 49.4284)
+			)
+		)
+	)
 	(embedded_fonts no)
