File: Amplifier.kicad_sch (KiCad schematic)
At the start: 22 parts, among them Q1 BC547, Q2 2N3904

Commit message: 2.26.2026
Other:
- title: Power Amplifier -> Amplifier
Changed lines of the file:
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@@
 	(paper "A4")
 	(title_block
-		(title "Power Amplifier")
+		(title "Amplifier")
 	)
 	(text "[ DESIGN SPECIFICATIONS ]\n-------------------------\nInput Signal (Vsig): 5mVrms\nTest Frequency:      1kHz\nLow Cutoff (fL):     80Hz\nHigh Cutoff (fH):    20kHz\nLoad (RL):           4k7"
